Commit message: Finished ASD assignment

File: src/gazebo/launch/robot.urdf (robot description, URDF)
Before this commit: robot robot, 4 links, 0 joints
Joints:
- added joint caster_joint: type fixed, parent robot/chassis, child robot/caster, origin xyz=0.8 0 -0.2 rpy=0 0 0
- added joint left_wheel_joint: type continuous, parent robot/chassis, child robot/left_wheel, origin xyz=-0.5 0.6 0 rpy=-1.5707 0 0, axis 0 0 1, limit effort=100 velocity=100
- added joint right_wheel_joint: type continuous, parent robot/chassis, child robot/right_wheel, origin xyz=-0.5 -0.6 0 rpy=-1.5707 0 0, axis 0 0 1, limit effort=100 velocity=100
